File: R_esc.kicad_sch (KiCad schematic)
At the start: 0 parts

Commit message: shema and footprints are mostly done
Parts:
- added C1: 4.7uF, Capacitor_SMD:C_0805_2012Metric, symbol Device:C
- added C10, C11, C12, C13: 1uF, Capacitor_SMD:C_0805_2012Metric, symbol Device:C
- added C2: 0.1uF, Capacitor_SMD:C_0603_1608Metric, symbol Device:C
- added C3, C5, C9: 10uF, Capacitor_SMD:C_1206_3216Metric, symbol Device:C
- added C4, C6: 22uF, Capacitor_SMD:C_1206_3216Metric, symbol Device:C
- added C7: 1nF, Capacitor_SMD:C_0603_1608Metric, symbol Device:C
- added C8: 100nF, Capacitor_SMD:C_0603_1608Metric, symbol Device:C
- added D1: SS34, Diode_SMD:D_SMA, symbol Diode:SS34
- added D2, D3, D4: 1N4148WT, Diode_SMD:D_SOD-523, symbol Diode:1N4148WT
- added D5: SMBJ30CA, SMBJ30CA:DIOM4336X265N, symbol SMBJ30CA:SMBJ30CA
- added J1: Conn_01x03_Pin, Connector_PinHeader_2.54mm:PinHeader_1x03_P2.54mm_Vertical, symbol Connector:Conn_01x03_Pin
- added J2: Conn_01x04_Pin, Connector_PinHeader_2.54mm:PinHeader_1x04_P2.54mm_Vertical, symbol Connector:Conn_01x04_Pin
- added J3, J4, J5, J6, J7: Conn_01x01_Pin, Connector_Wire:SolderWirePad_1x01_SMD_5x10mm, symbol Connector:Conn_01x01_Pin
- added L1: 22uH, Inductor_SMD:L_6.3x6.3_H3, symbol Device:L
- added NT1: NetTie_2, NetTie:NetTie-2_SMD_Pad0.5mm, symbol Device:NetTie_2
- added R1: 100K, Resistor_SMD:R_0603_1608Metric, symbol Device:R
- added R10, R11, R12, R13, R14, R9: 0.02k, Resistor_SMD:R_0603_1608Metric, symbol Device:R
- added R15, R16, R17, R18, R19, R2, R20, R7, R8: 10K, Resistor_SMD:R_0603_1608Metric, symbol Device:R
- added R21, R24, R27: 10k, Resistor_SMD:R_0603_1608Metric, symbol Device:R
- added R22, R25, R28: 4.7k, Resistor_SMD:R_0603_1608Metric, symbol Device:R
- added R23, R29: 47k, Resistor_SMD:R_0603_1608Metric, symbol Device:R
- added R26: 47K, Resistor_SMD:R_0603_1608Metric, symbol Device:R
- added R3: 0.056k, Resistor_SMD:R_0603_1608Metric, symbol Device:R
- added R30, R31: 0.1K, Resistor_SMD:R_0603_1608Metric, symbol Device:R
- added R32: 1mR, Resistor_SMD:R_2512_6332Metric, symbol Device:R
- added R4: 100k, Resistor_SMD:R_0603_1608Metric, symbol Device:R
- added R5: 39k, Resistor_SMD:R_0603_1608Metric, symbol Device:R
- added R6: 3.3K, Resistor_SMD:R_0603_1608Metric, symbol Device:R
- added U1: STM32F051K8U6, STM32F051K8U6:QFN50P500X500X60-33N, symbol STM32F051K8U6:STM32F051K8U6
- added U10, U5, U6, U7, U8, U9: SQJ138ELP-T1_GE3, footprints_5:PowerPAK_SO-8L_3_VIS, symbol 2026-02-16_08-09-54:SQJ138ELP-T1_GE3
- added U2: INA199A1DCKR, INA199A1DCKR:SOT65P210X110-6N, symbol INA199A1DCKR:INA199A1DCKR
- added U3: AOZ1282CI, Package_TO_SOT_SMD:SOT-23-6, symbol Regulator_Switching:AOZ1282CI
- added U4: AMS1117-3.3, Package_TO_SOT_SMD:SOT-223-3_TabPin2, symbol Regulator_Linear:AMS1117-3.3
- added driver1: FD6288Q, footprints_4:QFN24_FOR-M, symbol 2026-02-15_08-33-50:FD6288Q
Connections:
- new net: C13.1, D2.1 (K), driver1.17 (VB2)
- new net: C12.1, D4.1 (K), driver1.20 (VB1)
- new net: R7.2, U1.31 (BOOT0)
- new net: R12.2, R18.1, U7.4 (G)
- new net: R15.1, R9.2, U5.4 (G)
- new net: C11.1, D3.1 (K), driver1.14 (VB3)
- new net: R3.1, U2.6 (OUT)
- new net: C2.1, U3.1 (BST)
- new net: R5.2, R6.1, U3.3 (FB)
- new net: R4.2, U3.4 (EN)
- new net: C2.2, L1.1, U3.6 (LX)
- new net: R14.2, R20.1, U9.4 (G)
- new net: R10.2, R16.1, U6.4 (G)
- new net: R30.2, U1.26 (PB3/SPI1_SCK/I2S1_CK/TIM2_CH2/TSC_G5_IO1/EVENTOUT)
- new net: R31.2, U1.29 (PB6/I2C1_SCL/USART1_TX/TIM16_CH1N/TSC_G5_IO3)
- new net: R8.2, U1.4 (NRST)
- new net: R11.2, R17.1, U8.4 (G)
- new net: R13.2, R19.1, U10.4 (G)
- new net +10v: C10.1, C3.1, C5.1, C9.1, D1.1 (K), D2.2 (A), D3.2 (A), D4.2 (A), L1.2, R5.1, U4.3 (VI), driver1.4 (VCC)
- new net ADC_Cur: R3.2, U1.9 (PA3/USART2_RX/TIM2_CH4/TIM15_CH2/TSC_G1_IO4/ADC_IN3/COMP2_INP)
- new net ADC_vcc: C8.2, R1.2, R2.2, U1.12 (PA6/SPI1_MISO/I2S1_MCK/TIM3_CH1/TIM1_BKIN/TIM16_CH1/COMP1_OUT/TSC_G2_IO3/EVENTOUT/ADC_IN6)
- new net BackEMF_A: R21.1, R22.2, R23.1, U1.6 (PA0/USART2_CTS/TIM2_CH1_ETR/COMP1_OUT/TSC_G1_IO1/ADC_IN0/COMP1_INM6/RTC_TAMP2/WKUP1)
- new net BackEMF_B: R24.1, R25.2, R26.1, U1.10 (PA4/SPI1_NSS/I2S1_WS/USART2_CK/TIM14_CH1/TSC_G2_IO1/ADC_IN4/COMP1_INM4/COMP2_INM4/DAC_OUT1)
- new net BackEMF_C: R27.1, R28.2, R29.1, U1.11 (PA5/SPI1_SCK/I2S1_CK/CEC/TIM2_CH1_ETR/TSC_G2_IO2/ADC_IN5/COMP1_INM5/COMP2_INM5)
- new net BackEMF_Ortak: R21.2, R24.2, R27.2, U1.8 (PA2/USART2_TX/TIM2_CH3/TIM15_CH1/COMP2_OUT/TSC_G1_IO3/ADC_IN2/COMP2_INM6)
- new net Motor1_A: C12.2, J3.1 (Pin_1), R15.2, R23.2, U5.1 (S), U5.2 (S), U5.3 (S), U6.5 (D), driver1.18 (VS1)
- new net Motor1_A_gatehigh: R9.1, driver1.19 (HO1)
- new net Motor1_A_gatelow: R10.1, driver1.11 (LO1)
- new net Motor1_B: C13.2, J4.1 (Pin_1), R18.2, R26.2, U7.1 (S), U7.2 (S), U7.3 (S), U8.5 (D), driver1.15 (VS2)
- new net Motor1_B_gatehigh: R12.1, driver1.16 (HO2)
- new net Motor1_B_gatelow: R11.1, driver1.10 (LO2)
- new net Motor1_C: C11.2, J5.1 (Pin_1), R20.2, R29.2, U10.5 (D), U9.1 (S), U9.2 (S), U9.3 (S), driver1.12 (VS3)
- new net Motor1_C_gatehigh: R14.1, driver1.13 (HO3)
- new net Motor1_C_gatelow: R13.1, driver1.9 (LO3)
- new net Motor1_HIGH_A: U1.20 (PA10/USART1_RX/TIM1_CH3/TIM17_BKIN/TSC_G4_IO2), driver1.22 (HIN1)
- new net Motor1_HIGH_B: U1.19 (PA9/USART1_TX/TIM1_CH2/TIM15_BKIN/TSC_G4_IO1), driver1.23 (HIN2)
- new net Motor1_HIGH_C: U1.18 (PA8/USART1_CK/TIM1_CH1/EVENTOUT/MCO), driver1.24 (HIN3)
- new net Motor1_LOW_A: U1.15 (PB1/TIM3_CH4/TIM14_CH1/TIM1_CH3N/TSC_G3_IO3/ADC_IN9), driver1.1 (LIN1)
- new net Motor1_LOW_B: U1.14 (PB0/TIM3_CH3/TIM1_CH2N/TSC_G3_IO2/EVENTOUT/ADC_IN8), driver1.2 (LIN2)
- new net Motor1_LOW_C: U1.13 (PA7/SPI1_MOSI/I2S1_SD/TIM3_CH2/TIM14_CH1/TIM1_CH1N/TIM17_CH1/COMP2_OUT/TSC_G2_IO4/EVENTOUT/ADC_IN7), driver1.3 (LIN3)
- new net SWCLK: J2.2 (Pin_2), U1.24 (PA14/USART2_TX/SWCLK)
- new net SWDIO: J2.3 (Pin_3), U1.23 (PA13/IR_OUT/SWDIO)
- new net Signalin: J1.1 (Pin_1), R30.1
- new net UART_TX: J1.2 (Pin_2), R31.1
- new net VDD: C4.1, C6.2, J2.1 (Pin_1), R8.1, U1.1 (VDD), U1.17 (VDD), U1.5 (VDDA), U2.3 (V+), U4.2 (VO)
- new net Vcc: C7.2, D5.2, J7.1 (Pin_1), R1.1, R32.1, U2.4 (IN+)
- new net Vcc_M: C1.1, C7.1, R32.2, R4.1, U2.5 (IN-), U3.5 (VIN), U5.5 (D), U7.5 (D), U9.5 (D)
- new net gnd_d: C10.2, C6.1, C9.2, J1.3 (Pin_3), J2.4 (Pin_4), NT1.2, R22.1, R25.1, R28.1, R7.1, U1.33 (VSS), driver1.6 (COM)
- new net gnd_p: C1.2, C3.2, C4.2, C5.2, C8.1, D1.2 (A), D5.1, J6.1 (Pin_1), NT1.1, R16.2, R17.2, R19.2, R2.1, R6.2, U10.1 (S), U10.2 (S), U10.3 (S), U2.1 (REF), U2.2 (GND), U3.2 (GND), U4.1 (GND), U6.1 (S), U6.2 (S), U6.3 (S), U8.1 (S), U8.2 (S), U8.3 (S), driver1.25 (EPAD)
- no-connect marks 0 -> 11
Other:
- note added: "10v regülatör"
- note added: "3.3v regülatör"
- note added: "Akım okuma"
- note added: "GATE DRİVER"
- note added: "KODLAMA"
- note added: "OTOPİLOT"
- note added: "gerilim okuma"
- note added: "çıkış"

Commit message: layout eklendi
Parts:
- J3, J4, J5, J6, J7: footprint Connector_Wire:SolderWirePad_1x01_SMD_5x10mm -> Connector_PinHeader_2.54mm:PinHeader_1x01_P2.54mm_Vertical
Connections:
- net Vcc: now also C1.1, R4.1, U3.5 (VIN)
- net Vcc_M: no longer C1.1, R4.1, U3.5 (VIN)
Changed lines of the file:
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@@
 	(wire
 		(pts
+			(xy 171.45 95.25) (xy 170.18 95.25)
+		)
+		(stroke
+			(width 0)
+			(type default)
+		)
+	)
+	(wire
+		(pts
 			(xy 165.1 182.88) (xy 167.64 182.88)
 		)
@@
 	(wire
 		(pts
+			(xy 170.18 95.25) (xy 170.18 93.98)
+		)
+		(stroke
+			(width 0)
+			(type default)
+		)
+	)
+	(wire
+		(pts
 			(xy 55.88 91.44) (xy 74.93 91.44)
 		)
@@
 	(wire
 		(pts
+			(xy 76.2 66.04) (xy 74.93 66.04)
+		)
+		(stroke
+			(width 0)
+			(type default)
+		)
+	)
+	(wire
+		(pts
 			(xy 245.11 190.5) (xy 247.65 190.5)
 		)
@@
 	(wire
 		(pts
-			(xy 170.18 95.25) (xy 170.18 93.98)
-		)
-		(stroke
-			(width 0)
-			(type default)
-		)
-	)
-	(wire
-		(pts
 			(xy 74.93 91.44) (xy 74.93 83.82)
 		)
@@
 	)
 	(label "3.3v"
-		(at 74.93 66.04 0)
+		(at 76.2 66.04 0)
 		(effects
 			(font
@@
 	)
 	(label "Motor1_B_gatehigh"
-		(at 170.18 95.25 0)
+		(at 171.45 95.25 0)
 		(effects
 			(font
@@
 		)
 	)
-	(global_label "Vcc_M"
+	(global_label "Vcc"
 		(shape input)
 		(at 27.94 175.26 90)
@@
 		)
 		(property "Intersheetrefs" "${INTERSHEET_REFS}"
-			(at 27.94 166.59 90)
+			(at 27.94 169.009 90)
 			(effects
 				(font
@@
 			)
 		)
-		(property "Footprint" "Connector_Wire:SolderWirePad_1x01_SMD_5x10mm"
+		(property "Footprint" "Connector_PinHeader_2.54mm:PinHeader_1x01_P2.54mm_Vertical"
 			(at 86.36 21.59 0)
 			(effects
@@
 			)
 		)
-		(property "Footprint" "Connector_Wire:SolderWirePad_1x01_SMD_5x10mm"
+		(property "Footprint" "Connector_PinHeader_2.54mm:PinHeader_1x01_P2.54mm_Vertical"
 			(at 368.3 149.86 0)
 			(effects
@@
 			)
 		)
-		(property "Footprint" "Connector_Wire:SolderWirePad_1x01_SMD_5x10mm"
+		(property "Footprint" "Connector_PinHeader_2.54mm:PinHeader_1x01_P2.54mm_Vertical"
 			(at 83.82 21.59 0)
 			(effects
@@
 			)
 		)
-		(property "Footprint" "Connector_Wire:SolderWirePad_1x01_SMD_5x10mm"
+		(property "Footprint" "Connector_PinHeader_2.54mm:PinHeader_1x01_P2.54mm_Vertical"
 			(at 368.3 144.78 0)
 			(effects
@@
 			)
 		)
-		(property "Footprint" "Connector_Wire:SolderWirePad_1x01_SMD_5x10mm"
+		(property "Footprint" "Connector_PinHeader_2.54mm:PinHeader_1x01_P2.54mm_Vertical"
 			(at 368.3 147.32 0)
 			(effects
