File: R_esc.kicad_pcb (KiCad board)
At the start: 4 copper layers, 61.6 x 35.8 mm, 70 parts, among them J1 Conn_01x03_Pin, J2 Conn_01x04_Pin, J3 Conn_01x01_Pin, J4 Conn_01x01_Pin, J5 Conn_01x01_Pin, J6 Conn_01x01_Pin, J7 Conn_01x01_Pin, U1 STM32F051K8U6, U10 SQJ138ELP-T1_GE3, U2 INA199A1DCKR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

Commit message: new commit
Parts:
- moved J6 31.9 mm to (147.8, 64.6)
Routing:
- net (no net): vias 34 -> 37
- added copper zone on F.Cu, net (none)
Other:
- board size 61.6 x 35.8 mm -> 61.6 x 35.9 mm
- board text added: "GND"
- board text added: "SIGNAL"
- board text added: "SWCLK"
- board text added: "SWDIO"
- board text added: "UART_TX"
- board text added: "VCC"
- board text added: "VDD"
Changed lines of the file:
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@@
 	(footprint "Connector_PinHeader_2.54mm:PinHeader_1x01_P2.54mm_Vertical"
 		(layer "F.Cu")
-		(at 169.164 88.392 90)
+		(at 147.85 64.6 90)
 		(descr "Through hole straight pin header, 1x01, 2.54mm pitch, single row")
 		(tags "Through hole pin header THT 1x01 2.54mm single row")
@@
 			(at 0 -2.38 90)
 			(layer "F.SilkS")
+			(hide yes)
 			(effects
 				(font
@@
 			(at 0 -2.38 90)
 			(layer "F.SilkS")
+			(hide yes)
 			(effects
 				(font
@@
 	(gr_poly
 		(pts
-			(xy 121.45 61.95) (xy 121.3 93.55) (xy 126.15 93.4) (xy 129.35 96.25) (xy 139.3 96.3) (xy 141 97.55)
-			(xy 148.8 97.45) (xy 182.9 97.7) (xy 182.6 61.9)
+			(xy 121.45 61.95) (xy 121.3 93.55) (xy 126.1872 93.5228) (xy 129.54 96.52) (xy 139.3 96.52) (xy 140.97 97.79)
+			(xy 149.2 97.7) (xy 182.9 97.7) (xy 182.6 61.9)
 		)
 		(stroke
@@
 		(layer "Edge.Cuts")
 	)
+	(gr_circle
+		(center 178.251472 95.4)
+		(end 178.851472 96)
+		(stroke
+			(width 0.05)
+			(type default)
+		)
+		(fill no)
+		(layer "Edge.Cuts")
+	)
+	(gr_text "UART_TX\n"
+		(at 129 72.7 0)
+		(layer "F.SilkS")
+		(effects
+			(font
+				(size 0.5 0.4)
+				(thickness 0.1)
+			)
+			(justify left bottom)
+		)
+	)
+	(gr_text "VCC"
+		(at 150.4 69.1 90)
+		(layer "F.SilkS")
+		(effects
+			(font
+				(size 0.5 0.5)
+				(thickness 0.1)
+			)
+			(justify left bottom)
+		)
+	)
+	(gr_text "GND\n"
+		(at 150.4 65.4 90)
+		(layer "F.SilkS")
+		(effects
+			(font
+				(size 0.5 0.5)
+				(thickness 0.1)
+			)
+			(justify left bottom)
+		)
+	)
+	(gr_text "SWDIO\n"
+		(at 130.4 65.3 0)
+		(layer "F.SilkS")
+		(effects
+			(font
+				(size 0.5 0.5)
+				(thickness 0.1)
+			)
+			(justify left bottom)
+		)
+	)
+	(gr_text "VDD\n"
+		(at 125.2 65.3 0)
+		(layer "F.SilkS")
+		(effects
+			(font
+				(size 0.5 0.5)
+				(thickness 0.1)
+			)
+			(justify left bottom)
+		)
+	)
+	(gr_text "GND\n"
+		(at 132 72.7 0)
+		(layer "F.SilkS")
+		(effects
+			(font
+				(size 0.5 0.5)
+				(thickness 0.1)
+			)
+			(justify left bottom)
+		)
+	)
+	(gr_text "GND\n"
+		(at 133.2 65.3 0)
+		(layer "F.SilkS")
+		(effects
+			(font
+				(size 0.5 0.5)
+				(thickness 0.1)
+			)
+			(justify left bottom)
+		)
+	)
+	(gr_text "SWCLK\n"
+		(at 127.5 65.3 0)
+		(layer "F.SilkS")
+		(effects
+			(font
+				(size 0.5 0.5)
+				(thickness 0.1)
+			)
+			(justify left bottom)
+		)
+	)
+	(gr_text "SIGNAL\n"
+		(at 126 72.7 0)
+		(layer "F.SilkS")
+		(effects
+			(font
+				(size 0.5 0.5)
+				(thickness 0.1)
+			)
+			(justify left bottom)
+		)
+	)
 	(via
-		(at 159.6 94.3)
+		(at 160.02 96.52)
 		(size 0.6)
 		(drill 0.3)
@@
 	)
 	(via
-		(at 159.4 93.2)
+		(at 172.72 93.98)
 		(size 0.6)
 		(drill 0.3)
@@
 	)
 	(via
-		(at 137.5 68.8)
+		(at 157.48 93.98)
 		(size 0.6)
 		(drill 0.3)
@@
 	)
 	(via
-		(at 136.5 68.85)
+		(at 181.61 92.71)
 		(size 0.6)
 		(drill 0.3)
@@
 	)
 	(via
-		(at 137.4 66.85)
+		(at 172.72 96.52)
 		(size 0.6)
 		(drill 0.3)
@@
 	)
 	(via
-		(at 181.1 93.15)
+		(at 137.16 67.31)
 		(size 0.6)
 		(drill 0.3)
@@
 	)
 	(via
-		(at 159.65 94.95)
+		(at 162.56 96.52)
 		(size 0.6)
 		(drill 0.3)
@@
 	)
 	(via
-		(at 138.35 66.85)
+		(at 160.02 93.98)
 		(size 0.6)
 		(drill 0.3)
@@
 	)
 	(via
-		(at 138.3 67.85)
+		(at 181.61 93.98)
 		(size 0.6)
 		(drill 0.3)
@@
 	)
 	(via
-		(at 159.65 95.75)
+		(at 175.26 93.98)
 		(size 0.6)
 		(drill 0.3)
@@
 	)
 	(via
-		(at 181 87.35)
+		(at 181.61 87.63)
 		(size 0.6)
 		(drill 0.3)
@@
 	)
 	(via
-		(at 137.55 67.85)
+		(at 181.61 91.44)
 		(size 0.6)
 		(drill 0.3)
@@
 	)
 	(via
-		(at 136.5 67.85)
+		(at 181.61 88.9)
 		(size 0.6)
 		(drill 0.3)
@@
 	)
 	(via
-		(at 156.6 92.3)
+		(at 154.94 96.52)
 		(size 0.6)
 		(drill 0.3)
@@
 	)
 	(via
-		(at 156.6 94.95)
+		(at 170.18 96.52)
 		(size 0.6)
 		(drill 0.3)
@@
 	)
 	(via
-		(at 136.5 66.85)
+		(at 181.61 95.25)
 		(size 0.6)
 		(drill 0.3)
@@
 	)
 	(via
-		(at 181.1 94.8)
+		(at 165.1 96.52)
 		(size 0.6)
 		(drill 0.3)
@@
 	)
 	(via
-		(at 181.1 92.2)
+		(at 167.64 96.52)
 		(size 0.6)
 		(drill 0.3)
@@
 	)
 	(via
-		(at 181.1 91.15)
+		(at 154.94 96.52)
 		(size 0.6)
 		(drill 0.3)
@@
 	)
 	(via
-		(at 156.6 95.75)
+		(at 138.43 68.58)
 		(size 0.6)
 		(drill 0.3)
@@
 	)
 	(via
-		(at 181.1 90.3)
+		(at 137.16 68.58)
 		(size 0.6)
 		(drill 0.3)
@@
 	)
 	(via
-		(at 162.1 95.8)
+		(at 139.7 67.31)
 		(size 0.6)
 		(drill 0.3)
@@
 	)
 	(via
-		(at 156.6 94.2)
+		(at 162.56 93.98)
 		(size 0.6)
 		(drill 0.3)
@@
 	)
 	(via
-		(at 181 88.35)
+		(at 157.48 96.52)
 		(size 0.6)
 		(drill 0.3)
@@
 	)
 	(via
-		(at 164.4 82.6)
+		(at 165.1 93.98)
 		(size 0.6)
 		(drill 0.3)
@@
 	)
 	(via
-		(at 156.6 93.25)
+		(at 138.43 67.31)
 		(size 0.6)
 		(drill 0.3)
@@
 	)
 	(via
-		(at 181.05 89.45)
+		(at 154.94 93.98)
 		(size 0.6)
 		(drill 0.3)
@@
 	)
 	(via
-		(at 166.65 84.65)
+		(at 181.61 90.17)
+		(size 0.6)
+		(drill 0.3)
+		(layers "F.Cu" "B.Cu")
+		(net 0)
+	)
+	(via
+		(at 164.4 82.6)
 		(size 0.6)
 		(drill 0.3)
@@
 	)
 	(via
-		(at 162.1 94.95)
+		(at 167.64 93.98)
+		(size 0.6)
+		(drill 0.3)
+		(layers "F.Cu" "B.Cu")
+		(net 0)
+	)
+	(via
+		(at 170.18 93.98)
+		(size 0.6)
+		(drill 0.3)
+		(layers "F.Cu" "B.Cu")
+		(net 0)
+	)
+	(via
+		(at 166.65 84.65)
 		(size 0.6)
 		(drill 0.3)
@@
 	)
 	(via
-		(at 161.95 93.3)
+		(at 175.26 96.52)
 		(size 0.6)
 		(drill 0.3)
@@
 	)
 	(via
-		(at 181.1 93.95)
+		(at 139.7 68.58)
 		(size 0.6)
 		(drill 0.3)
@@
 	)
 	(via
-		(at 162.05 94.2)
+		(at 181.61 96.52)
 		(size 0.6)
 		(drill 0.3)
@@
 			)
 		)
+	)
+	(zone
+		(net 0)
+		(net_name "")
+		(layer "F.Cu")
+		(hatch edge 0.5)
+		(priority 8)
+		(connect_pads
+			(clearance 0.5)
+		)
+		(min_thickness 0.25)
+		(filled_areas_thickness no)
+		(fill yes
+			(thermal_gap 0.5)
+			(thermal_bridge_width 0.5)
+			(island_removal_mode 1)
+			(island_area_min 10)
+		)
+		(polygon
+			(pts
+				(xy 121.92 62.23) (xy 122.2248 92.6592) (xy 127 92.6592) (xy 129.54 95.25) (xy 139.7 95.25) (xy 140.97 96.52)
+				(xy 181.61 96.52) (xy 181.61 62.23)
+			)
+		)
